File: Kicad/V1/Illustrabot2_IF_Motor_Beagle_v1.kicad_pcb (KiCad board)
At the start: 2 copper layers, 0 parts

Commit message: Footprint association Component placing
Parts:
- added C1: 100uF, CP4, F.Cu at (64.8, 188.0)
- added C10: 100nF, C1, F.Cu at (153.7, 163.8)
- added C11: 100uF, CP4, F.Cu at (212.1, 188.0)
- added C12: 100uF, CP4, F.Cu at (101.6, 188.0)
- added C13: 100nF, C1, F.Cu at (264.2, 163.8)
- added C14: 100nF, C1, F.Cu at (116.8, 163.8)
- added C2: 100uF, CP4, F.Cu at (175.3, 188.0)
- added C3: 10uF, C1, F.Cu at (74.9, 111.8)
- added C4: 10uF, C1, F.Cu at (78.7, 87.6)
- added C5: 100nF, C1, F.Cu at (80.0, 163.8)
- added C6: 100nF, C1, F.Cu at (190.5, 163.8)
- added C7: 100uF, CP4, F.Cu at (248.9, 188.0)
- added C8: 100uF, CP4, F.Cu at (138.4, 188.0)
- added C9: 100nF, C1, F.Cu at (227.3, 163.8)
- added D1: LED, LED-3MM, F.Cu at (119.4, 58.4)
- added D2: LED, LED-3MM, F.Cu at (134.6, 58.4)
- added D3: LED, LED-3MM, F.Cu at (151.1, 58.4)
- added D4: LED, LED-3MM, F.Cu at (166.4, 58.4)
- added D5: LED, LED-3MM, F.Cu at (181.6, 58.4)
- added D6: LED, LED-3MM, F.Cu at (198.1, 59.7)
- added JP1: JUMPER3, SIL-3, F.Cu at (77.5, 99.1)
- added JP2: JUMPER, SIL-2, F.Cu at (72.4, 163.8)
- added JP3: JUMPER, SIL-2, F.Cu at (182.9, 163.8)
- added JP4: JUMPER, SIL-2, F.Cu at (219.7, 163.8)
- added JP5: JUMPER, SIL-2, F.Cu at (146.1, 163.8)
- added JP6: JUMPER, SIL-2, F.Cu at (256.5, 163.8)
- added JP7: JUMPER, SIL-2, F.Cu at (109.2, 163.8)
- added P1: CONN_4, bornier4, F.Cu at (80.0, 198.1)
- added P10: CONN_4, bornier4, F.Cu at (181.6, 35.6)
- added P11: CONN_4, bornier4, F.Cu at (129.5, 35.6)
- added P12: CONN_4, bornier4, F.Cu at (116.8, 198.1)
- added P2: CONN_4, bornier4, F.Cu at (190.5, 198.1)
- added P3: CONN_4, bornier4, F.Cu at (61.0, 106.7)
- added P4: CONN_4, bornier4, F.Cu at (292.1, 177.8)
- added P5: CONN_4, bornier4, F.Cu at (227.3, 198.1)
- added P6: CONN_4, bornier4, F.Cu at (153.7, 198.1)
- added P7: CONN_4, bornier4, F.Cu at (264.2, 198.1)
- added P8: CONN_23X2, SIL-2x23-v1, F.Cu at (165.1, 130.8)
- added P9: CONN_23X2, SIL-2x23-v1, F.Cu at (165.1, 82.5)
- added Q1: NPN, TO92, F.Cu at (128.3, 66.0)
- added Q2: NPN, TO92, F.Cu at (144.8, 66.0)
- added Q3: NPN, TO92, F.Cu at (160.0, 66.0)
- added Q4: NPN, TO92, F.Cu at (175.3, 67.3)
- added Q5: NPN, TO92, F.Cu at (190.5, 67.3)
- added Q6: NPN, TO92, F.Cu at (208.3, 67.3)
- added R1: 10kohm, R3, F.Cu at (81.3, 154.9)
- added R10: 10kohm, R3, F.Cu at (265.4, 156.2)
- added R11: 82kohm, R3, F.Cu at (158.8, 49.5)
- added R12: 10kohm, R3, F.Cu at (118.1, 156.2)
- added R13: 150ohm, R3, F.Cu at (166.4, 49.5)
- added R14: 82kohm, R3, F.Cu at (174.0, 49.5)
- added R15: 150ohm, R3, F.Cu at (181.6, 49.5)
- added R16: 82kohm, R3, F.Cu at (189.2, 49.5)
- added R17: 150ohm, R3, F.Cu at (198.1, 49.5)
- added R18: 82kohm, R3, F.Cu at (207.0, 49.5)
- added R19: 10kohm, R3, F.Cu at (73.7, 154.9)
- added R2: 10kohm, R3, F.Cu at (191.8, 156.2)
- added R20: 10kohm, R3, F.Cu at (184.2, 156.2)
- added R21: 10kohm, R3, F.Cu at (221.0, 156.2)
- added R22: 10kohm, R3, F.Cu at (147.3, 156.2)
- added R23: 10kohm, R3, F.Cu at (257.8, 156.2)
- added R24: 10kohm, R3, F.Cu at (110.5, 156.2)
- added R3: 10kohm, R3, F.Cu at (228.6, 156.2)
- added R4: 10kohm, R3, F.Cu at (154.9, 156.2)
- added R5: 150ohm, R3, F.Cu at (119.4, 49.5)
- added R6: 82kohm, R3, F.Cu at (127.0, 49.5)
- added R7: 150ohm, R3, F.Cu at (134.6, 49.5)
- added R8: 82kohm, R3, F.Cu at (143.5, 49.5)
- added R9: 150ohm, R3, F.Cu at (151.1, 49.5)
- added U1: STEPSTICK, Stepstick_footprint, F.Cu at (80.0, 176.5)
- added U2: STEPSTICK, Stepstick_footprint, F.Cu at (190.5, 176.5)
- added U3: STEPSTICK, Stepstick_footprint, F.Cu at (227.3, 176.5)
- added U4: STEPSTICK, Stepstick_footprint, F.Cu at (153.7, 176.5)
- added U5: STEPSTICK, Stepstick_footprint, F.Cu at (264.2, 176.5)
- added U6: STEPSTICK, Stepstick_footprint, F.Cu at (116.8, 176.5)
Routing:
- net GND: track 0.00 -> 203.2 mm
- net 3V3: track 0.00 -> 45.7 mm
- net N-0000081: track 0.00 -> 20.3 mm
- net N-0000083: track 0.00 -> 19.1 mm
- net N-0000080: track 0.00 -> 19.0 mm
- net N-0000082: track 0.00 -> 19.0 mm
- net N-000008: track 0.00 -> 19.0 mm
- net N-0000068: track 0.00 -> 19.0 mm
- net /2B_M6: track 0.00 -> 16.8 mm
- net /2B_M5: track 0.00 -> 16.8 mm
- net /2B_M4: track 0.00 -> 16.8 mm
- net /2B_M3: track 0.00 -> 16.8 mm
- net /2B_M2: track 0.00 -> 16.8 mm
- net /2B_M1: track 0.00 -> 16.8 mm
- net /1B_M5: track 0.00 -> 16.8 mm
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Other:
- net class 12V_12A added: clearance 0.31, trace_width 2, via_dia 0.889, via_drill 0.635
- net class 12V_2A added: clearance 0.31, trace_width 0.6, via_dia 0.889, via_drill 0.635
- net class Default: clearance 0.254 -> 0.31; trace_width 0.254 -> 0.31
- rule trace_clearance: 0.254 -> 0.31
- board text added: "Ne pas oublier les éléments suivants : empreinte vis fixation beaglebone empreinte vis carte fille zone interdite emplacement connecteur beaglebone + usblte"
