File: Kicad/V1/Illustrabot2_IF_Motor_Beagle_v1.kicad_pcb (KiCad board)
At the start: 2 copper layers, 73 parts, among them P1 CONN_4, P10 CONN_4, P11 CONN_4, P12 CONN_4, P13 CONN_1, P14 CONN_1, P15 CONN_1, P16 CONN_1, P2 CONN_4, P3 CONN_4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

Commit message: Final routing
Parts:
- moved JP1 32.9 mm to (56.5, 27.3)
- moved P3 32.9 mm to (40.0, 29.8)
- moved C4 30.5 mm to (55.2, 22.2)
- moved C7 21.7 mm to (250.8, 170.8)
- moved C10 21.7 mm to (126.4, 145.4)
- moved P6 21.7 mm to (126.4, 181.0)
- moved U4 21.7 mm to (126.4, 159.4)
- moved C1 21.7 mm to (66.7, 170.8)
- moved C11 21.7 mm to (214.0, 170.8)
- moved C12 21.7 mm to (103.5, 170.8)
- moved C13 21.7 mm to (236.9, 145.4)
- moved C14 21.7 mm to (89.5, 144.8)
- moved C15 21.7 mm to (41.9, 172.7)
- moved C16 21.7 mm to (152.4, 172.7)
- moved C17 21.7 mm to (189.2, 172.7)
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Routing:
- net GND: track 1506.3 -> 1409.3 mm
- net 3V3: track 1009.7 -> 1096.9 mm
- net GNDA: track 434.5 -> 409.6 mm
- net +12C: track 384.4 -> 360.6 mm
- net +5V: track 48.8 -> 26.7 mm
- net +12V: track 257.4 -> 238.3 mm
- net AGND: track 288.6 -> 276.1 mm
- net /Beaglebone_5V: track 60.9 -> 72.7 mm
- net N-0000036: track 23.8 -> 34.2 mm
- net /Direction_m6: track 170.4 -> 179.8 mm
- net /Step_m6: track 169.3 -> 178.1 mm
- net /direction_m1: track 92.0 -> 84.5 mm
- net /Step_m1: track 92.0 -> 84.9 mm
- net /Direction_m2: track 62.8 -> 55.8 mm
- net /Step_m2: track 62.8 -> 56.2 mm
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Other:
- net class 12V_2A: clearance 0.31 -> 0.8; trace_width 0.6 -> 0.8
- net class 12V_6A: clearance 0.45 -> 0.8
- net class Default: clearance 0.31 -> 0.6; trace_width 0.31 -> 0.8
- rule trace_clearance: 0.31 -> 0.6

Commit message: Modification P9 header (pin 25 -> pin 27)
Connections:
- P9 pad 25: /Position_m6 -> (no net)
- P9 pad 27: (no net) -> /Position_m6
Routing:
- net /Position_m6: track 56.2 -> 53.6 mm
